File: PublicSecurity96/PublicSecurity96.kicad_sch (KiCad schematic)
At the start: 239 parts, among them J1 USB_C_Receptacle_USB2.0, U1 XC6206PxxxMR, U2 SRV05-4, U3 RP2040, Y1 16MHz

Commit message: wip: U1 swap XC6206->AMS1117-3.3, bump LDO caps to 10uF
Schematic edits done in KiCad GUI:
- U1: Regulator_Linear:AMS1117-3.3 (was XC6206PxxxMR), JLCPCB C6186
- LDO input + output caps: 1uF -> 10uF for AMS1117 stability
- Added JLCPCB part# custom field column
- Started placing PWR_FLAG (+5V done, +3V3 in progress — wires off-grid)

ERC state: 3 errors (power_pin_not_driven, fixing with PWR_FLAGs)
+ 829 cosmetic off-grid warnings (legacy from copy-paste schematic).
PCM_marbastlib-mx still missing — install via PCM after restart.

Co-Authored-By: Claude Opus 4.7 <noreply@anthropic.com>
Parts:
- C1, C2: value 1uF -> 10uF; footprint Capacitor_SMD:C_0402_1005Metric_Pad0.74x0.62mm_HandSolder -> Capacitor_SMD:C_0805_2012Metric; JLCPCB# (none) -> C15850
- U1: footprint Package_TO_SOT_SMD:SOT-23-3 -> Package_TO_SOT_SMD:SOT-223-3_TabPin2; JLCPCB part# C47374 -> C15850
- renumbered C2 to C8, C1 to C9, H4 to H3, H5 to H4, H1 to H5, H2 to H6, H1 to H7, R6 to R4, R7 to R5, R8 to R6
